File: hardware/prototype/cinamin.sch (EAGLE design)
At the start: 93 parts, among them J1 TC2030-JLINK-L, Q1 MOSFET-NCHANNELXFDN-3, Q2 MOSFET-NCHANNELXFDN-3, Q5 MOSFET-NCHANNELXFDN-3, U1 ADM8641, U11 ADM8641, U2 ADM8641, U3 BQ25504RGT

Commit message: most of the way through layout
Parts:
- added R16: 2.2k, passives:RESISTOR0402_RES
- added RESET: B3U-1000P, switches:B3U-1000P
- added TP3, TP4, TP5, TP6, TP7, TP8: TPSPAD1-13, testpad:TPSPAD1-13
- JP22: value (none) -> TO_BLE
- JP24: value (none) -> TO_BQ25504
- TP1, TP2: value TPSQB1,27 -> TPSPAD1-13; device testpad:TPSQB1,27 -> testpad:TPSPAD1-13
- renumbered JP21 to SOLAR_TO_BQ, JP23 to PV_TO_CAPS, U$10 to U5, U$11 to SUPPLY_SELECTOR, U$12 to U7, U$13 to Q13, U$5 to U4, U$6 to U9, U$8 to U8, U11 to U6
Connections:
- removed net N$48: C14.2, R18.1, R21.1
- new net HIGH: JP20.1, Q10.D
- new net N$52: J1.SWDIO, U9.SWDIO
- new net N$53: J1.SWDCLK, U9.SW_CLK
- new net N$56: R16.2, RESET.P$1, U9.RST
- new net OUT: JP2.1, R3.1, U4.OUT
- new net OUT2: JP22.1, Q13.D
- new net VDD: JP19.2, Q10.S, U7.VDD
- new net VIN_DC: JP24.2, U3.VIN_DC
- new net VSTOR: C12.1, C13.1, Q13.S, U3.VOC_SAMP, U3.VSTOR
- net 580_VBAT: now also J1.VCC, RESET.P$2; no longer C12.1, C13.1, JP2.1, JP20.1, JP22.1, Q10.D, Q13.D, Q13.S, R3.1, U3.VOC_SAMP, U3.VSTOR, U4.OUT
- net AP4400: no longer JP19.2, Q10.S, U7.VDD
- net GND: now also C14.2, J1.GND, R16.1, R18.1, R21.1, TP2.PP, TP6.PP, TP7.PP, TP8.PP; no longer TP2.TP
- net N$43: now also TP1.PP, TP3.PP, TP4.PP, TP5.PP; no longer TP1.TP
- net PV: no longer JP24.2, U3.VIN_DC
Other:
- moved on the sheet: J1

Commit message: layout and schematic done
Parts:
- removed JP10: INPUT_DIVIDER, SparkFun-Passives:JUMPER-2PTH
- removed U$7: AF212M, chips:AF212M
- added A1: (no value), chips:AH212M
- added PROG: TC2030-JLINK-L, connector:TC2030-JLINK-L
- J1: value TC2030-JLINK-L -> INPUT_DIVIDER; device connector:TC2030-JLINK-L -> SparkFun-Passives:JUMPER-2PTH
- R1, R4: value (none) -> 2.2M
- R10, R11, R12, R13, R14, R15, R6, R7, R8, R9: value (none) -> 1M
- R2, R5: value (none) -> 1.18M
- R3: value (none) -> 3M
- U1: value ADM8641 -> 3.048
- U2: value ADM8641 -> 2.3
- renumbered JP1 to J18, JP11 to J2, JP12 to J15, JP13 to J12, JP14 to J13, JP15 to J14, JP16 to J11, JP17 to J16, JP18 to J17, JP19 to J19, JP2 to J3, JP20 to J20, JP22 to J22, JP24 to J21, JP3 to J10, JP4 to J5, JP5 to J4, JP6 to J7, JP7 to J8, JP8 to J6, JP9 to J9, U$1 to D4, U$2 to D3, U$3 to D2, U$4 to D1
Connections:
- removed net N$13: C10.1, C9.1, L2.2, U8.VDCDC, U8.VDCDC_RF
- new net N$48: X2.1
- new net N$55: U8.VDCDC
- new net N$57: C10.1
- new net N$58: C9.1
- net 580_VBAT: now also PROG.VCC; no longer J1.VCC
- net ADM8641_2: now also SUPPLY_SELECTOR.8; no longer SUPPLY_SELECTOR.12
- net BQ25504: now also SUPPLY_SELECTOR.12; no longer SUPPLY_SELECTOR.8
- net GND: now also PROG.GND; no longer C10.2, C8.2, C9.2, J1.GND, U8.GND, U8.RFIOM, U8.VBAT1V, X2.GND
- net LTC1540_I_HYST: now also J1.2; no longer JP10.2
- net N$12: no longer U8.SWITCH
- net N$16: no longer U8.XTAL16MP
- net N$17: no longer X2.1
- net N$27: now also J1.1; no longer JP10.1
- net N$5: now also A1.ANTENNA; no longer U$7.ANTENNA
- net N$52: now also PROG.SWDIO; no longer J1.SWDIO
- net N$53: now also PROG.SWDCLK; no longer J1.SWDCLK
- net N$6: now also U8.VDCDC_RF; no longer C8.1, U$9.ANTENNA, U8.RFIOP

Commit message: added series parrallel solar jumps
Parts:
- removed PV_TO_CAPS: FOR_BQ25504, SparkFun-Passives:JUMPER-2PTH
- removed SOLAR_TO_BQ: TO_BQ25504, SparkFun-Passives:JUMPER-2PTH
- added D1-2S, D2-3S, D3-4S: SER, SparkFun-Passives:JUMPER-2PTH
- added D1G, D2G, D3G, D4G: GND, SparkFun-Passives:JUMPER-2PTH
- added D1PV, D2PV, D3PV: HIGH, SparkFun-Passives:JUMPER-2PTH
- added PV_TO_CAP: (no value), SparkFun-Connectors:M03PTH
- added R17: 5.23M, passives:RESISTOR0402_RES
- added R23: 1.43M, passives:RESISTOR0402_RES
- added R24: 2.87M, passives:RESISTOR0402_RES
- added R25: 715k, passives:RESISTOR0402_RES
- added R26: 1.47M, passives:RESISTOR0402_RES
- A1: value (none) -> AH212M
- A2: value AF212M -> AH212M
- C1: value 100uF -> 15uF; device passives:CAP_POL0603 -> passives:CAPACITOR
- C10: value 1uF -> 100nF; device passives:CAPACITOR01005_CAP -> passives:CAPACITOR
- C11: value 4.7uF -> 1pF
- C12: value 0.1uF -> 1uF; device passives:CAPACITOR -> passives:CAPACITOR01005_CAP
- C13: value 4.7uF -> 100nF; device passives:CAPACITOR -> passives:CAPACITOR01005_CAP
- C14: value .01uF -> 1pF; device passives:CAPACITOR -> passives:CAPACITOR0201_CAP
- C2: value 1uF -> 15uF
- C3, C4: value 15uF -> 100uF; device passives:CAPACITOR -> passives:CAP_POL0603
- C5: value 100nF -> 4.7uF
- C6: value 100uF -> .01uF; device passives:CAP_POL0603 -> passives:CAPACITOR
- C7: value 1pF -> 0.1uF
- C8: value 1pF -> 4.7uF; device passives:CAPACITOR0201_CAP -> passives:CAPACITOR
- C9: value 100nF -> 1uF; device passives:CAPACITOR01005_CAP -> passives:CAPACITOR
- D1, D2, D3, D4: value (none) -> CPC1822
- J12: value STAGE_1_PULL -> INPUT_DIVIDER
- J13: value STAGE_2_PULL -> TO_LTC1540
- J14: value OFF_DIVIDER -> STAGE_1_PULL
- J15: value TO_BLE -> TO_AP440
- J16: value TO_ADM2 -> STAGE_2_PULL
- J17: value TO_ADM1 -> OFF_DIVIDER
- J2: value TO_LTC1540 -> (none)
- J20: value TO_AP440 -> TO_BLE
- J3: value TO_BLE -> TO_ADM2
- J4: value INPUT_DIVIDER -> TO_ADM1
- J5: value (none) -> TO_LATCH
- J6: value TO_LATCH -> STAGE_1_PULL
- J7: value STAGE_1_PULL -> STAGE_2_PULL
- J8: value STAGE_2_PULL -> OFF_DIVIDER
- J9: value OFF_DIVIDER -> TO_BLE
- L1: value 2.2uH -> 22uH; device passives:INDUCTOR0402 -> passives:INDUCTOR0603
- L2: value (none) -> 2.2uH
- L3: value 22uH -> 2.2uH; device passives:INDUCTOR0603 -> passives:INDUCTOR0402
- Q1: value MOSFET-NCHANNELXFDN-3 -> (none); device fets:MOSFET-NCHANNELXFDN-3 -> fets:MOSFET-PCHANNEL
- Q8: value (none) -> MOSFET-NCHANNELXFDN-3; device fets:MOSFET-PCHANNEL -> fets:MOSFET-NCHANNELXFDN-3
- R10: value 1M -> 1.18M
- R13: value 1M -> 3M
- R16: value 2.2k -> 4.87M
- R18: value 3.67M -> 3.24M
- R19: value 3.088M -> 3.09M
- R20: value 3.23M -> 3.65M
- R21: value 5.2M -> 2.2k
- R22: value 4.8M -> 3.48M
- R3: value 3M -> 1M
- R4: value 2.2M -> 1M
- R5: value 1.18M -> 1M
- R9: value 1M -> 2.2M
- U1: value 3.048 -> LTC1540; device chips:ADM8641 -> chips:LTC1540
- U2: value 2.3 -> (none); device chips:ADM8641 -> chips:ADM8642
- U3: value BQ25504RGT -> (none); device chips:BQ25504RGT -> chips:ADM8642
- U4: value U1 -> (none); device chips:LTC1540 -> chips:ADM8642
- U5: value U1 -> ltc1540
- U6: value ADM8641 -> AP4400_3.4_2.3; device chips:ADM8641 -> chips:AP4400
- U7: value (none) -> BQ25504RGT; device chips:AP4400 -> chips:BQ25504RGT
- U8: value (none) -> DA14580; device chips:DA14580-BGA -> chips:DA14580-48
- U9: device chips:DA14580-48 -> chips:DA14580-BGA
- X1, X2: value (none) -> 16Mhz
- renumbered Q13 to Q11, U$9 to A2
Connections:
- removed net N$18 (its old number): J4.1, R4.2
- removed net N$26 (its old number): J9.1, R8.2
- removed net N$4 (its old number): U4.HYST, U4.IN-, U4.REF
- new net N$13: J11.1, R22.2
- new net N$2: U1.HYST, U1.IN-, U1.REF
- new net N$21: J6.1, R4.2
- new net N$27: J12.1, R9.2
- new net N$59: R22.1, R23.2, U4.VIN
- new net N$60: R25.1, R26.2, U2.VIN
- new net N$61: D1.V-, D1G.2
- new net N$62: D1-2S.2, D2.V-, D2G.2
- new net N$63: D2-3S.2, D3.V-, D3G.2
- new net N$65: D1-2S.1, D1.V+, D1PV.2
- new net N$66: D1PV.1, D2PV.1, D3PV.1, D4.V+, PV_TO_CAP.2, TP1.PP, TP3.PP, TP4.PP, TP5.PP
- new net N$67: D2-3S.1, D2.V+, D2PV.2
- new net N$68: D3-4S.1, D3.V+, D3PV.2
- net 580_VBAT: now also J19.2, J9.2, U8.VBAT3V, U8.VBAT_RF; no longer J15.2, J3.2, U9.VBAT3V, U9.VBAT_RF
- net ADM8641: now also J14.2, J16.2, Q9.S, U4.VCC; no longer J12.2, J13.2, Q7.S
- net ADM8641_2: now also J3.2, J4.1; no longer J16.2, J17.1
- net AP4400: now also J15.1; no longer J19.1
- net BQ25504: now also U7.VBAT; no longer U3.VBAT
- net GND: now also C1.2, C10.2, C3.ANODE, C4.ANODE, C6.2, C8.2, C9.2, D1G.1, D2G.1, D3G.1, D4G.1, Q7.D, Q8.S, R10.1, R15.1, R17.1, R20.1, R23.1, R26.1, R3.1, R8.1, U1.V-, U8.GND, U8.GND1, U8.RFIOM, U8.VBAT1V; no longer C1.ANODE, C12.2, C13.2, C14.2, C3.2, C4.2, C6.ANODE, D1.V-, D2.V-, D3.V-, D4.V-, Q1.S, Q6.D, R13.1, R14.1, R16.1, R18.1, R5.1, R9.1, U4.V-, U9.GND, U9.GND1, U9.RFIOM, U9.VBAT1V
- net HIGH: now also J19.1; no longer J20.1
- net LTC1540_E_HYST: now also J1.2, J2.2, J5.1; no longer J4.2, J5.2, J6.1
- net LTC1540_I_HYST: now also J12.2, J13.1; no longer J1.2, J2.1
- net N$1: now also C1.1, C2.1, C3.CATHODE, C4.CATHODE, PV_TO_CAP.3; no longer C1.CATHODE, C3.1, C4.1, C6.CATHODE, PV_TO_CAPS.2
- net N$10: now also U8.XTAL16MP; no longer U9.XTAL16MP
- net N$11: now also U8.XTAL16MM; no longer U9.XTAL16MM
- net N$12: now also L3.1; no longer L2.1
- net N$14: now also R1.1, R2.2, U1.IN+; no longer R4.1, R5.2, U5.IN+
- net N$15: now also Q2.D, R4.1; no longer Q1.D, R6.1
- net N$17: now also U9.XTAL16MM; no longer U8.XTAL16MM
- net N$19: now also Q5.D, Q6.G, R6.1; no longer Q2.D, Q4.G, R7.1
- net N$20: now also J2.1, U1.V+; no longer J5.1, U5.V+
- net N$23: now also Q5.G, R7.1, R8.2; no longer Q2.G, R8.1, R9.2
- net N$24: now also J8.2, Q6.D; no longer J9.2, Q4.D
- net N$25: now also J5.2, Q6.S; no longer J8.2, Q4.S
- net N$28: now also J13.2, U5.V+; no longer J2.2, U4.V+
- net N$29: now also Q7.G, R11.1, U4.OUT; no longer Q6.G, R10.1, U6.OUT
- net N$3: now also R10.2, R13.2, R9.1, U5.IN+; no longer R1.1, R2.2, R3.2, U4.IN+
- net N$30: now also Q7.S, Q8.D, Q9.G, R12.1; no longer Q5.D, Q6.S, Q7.G, R11.1
- net N$31: now also Q8.G, R14.1, R15.2; no longer Q5.G, R12.1, R13.2
- net N$32: now also J17.2, J20.1, Q9.D; no longer J14.2, J15.1, Q7.D
- net N$33: now also J14.1, R11.2; no longer J12.1, R10.2
- net N$34: now also J16.1, R12.2; no longer J13.1, R11.2
- net N$35: now also R24.1, R25.2, U3.VIN; no longer J11.1, U6.VCC
- net N$36: now also J17.1, R14.2; no longer J14.1, R12.2
- net N$37: now also U6.DETOUT; no longer U7.DETOUT
- net N$38: now also J9.1, Q4.D; no longer J18.1, Q9.D
- net N$39: now also Q1.D, R3.2, U3.!DIS; no longer Q8.D, R14.2, U2.!DIS
- net N$40: now also J3.1, Q1.S, U3.VCC; no longer J16.1, Q8.S, U2.VCC
- net N$41: now also Q1.G, Q4.G, R5.1, U3.OUT; no longer Q8.G, Q9.G, R15.1, U1.OUT
- net N$42: now also J4.2, Q4.S, R24.2, R5.2, U2.VCC; no longer J17.2, Q9.S, R15.2, U1.VCC
- net N$43: now also D3-4S.2, D4.V-, D4G.2; no longer D1.V+, D2.V+, D3.V+, D4.V+, PV_TO_CAPS.1, SOLAR_TO_BQ.1, TP1.PP, TP3.PP, TP4.PP, TP5.PP
- net N$44: now also L1.1, U7.LBST, U7.OT_PROG; no longer L3.1, U3.LBST, U3.OT_PROG
- net N$45: now also U7.VBAT_UV; no longer U3.VBAT_UV
- net N$46: now also R16.2, R18.2, U7.VRDIV; no longer R20.2, R22.2, U3.VRDIV
- net N$47: now also U7.VBAT_OK; no longer U3.VBAT_OK
- net N$49: now also R18.1, U7.OK_HYST; no longer R20.1, U3.OK_HYST
- net N$5: now also C11.1, U8.RFIOP; no longer C7.1, U9.RFIOP
- net N$50: now also R20.2, U7.OK_PROG; no longer R18.2, U3.OK_PROG
- net N$51: now also C6.1, U7.VREF_SAMP; no longer C14.1, U3.VREF_SAMP
- net N$52: now also U8.SWDIO; no longer U9.SWDIO
- net N$53: now also U8.SW_CLK; no longer U9.SW_CLK
- net N$54: now also R16.1, R17.2, U7.VBAT_OV; no longer R21.2, R22.1, U3.VBAT_OV
- net N$55: now also U9.VDCDC; no longer U8.VDCDC
- net N$56: now also R21.2, U8.RST; no longer R16.2, U9.RST
- net N$57: now also C12.1; no longer C10.1
- net N$58: now also C13.1; no longer C9.1
- net N$6: now also U9.VDCDC_RF; no longer U8.VDCDC_RF
- net N$7: now also L2.1, U8.SWITCH; no longer L1.1, U9.SWITCH
- net N$8: now also C10.1, C9.1, L2.2, U8.VDCDC, U8.VDCDC_RF; no longer C2.1, C5.1, L1.2, U9.VDCDC, U9.VDCDC_RF
- net N$9: now also Q2.G, U1.OUT; no longer Q1.G, U5.OUT
- net OUT: now also J18.1, R13.1, U5.OUT; no longer J3.1, R3.1, U4.OUT
- net PV: now also C5.1, L1.2, PV_TO_CAP.1; no longer C11.1, L3.2, SOLAR_TO_BQ.2
- net VDD: now also J15.2, U6.VDD; no longer J19.2, U7.VDD
- net VIN_DC: now also U7.VIN_DC; no longer U3.VIN_DC
- net VSTOR: now also C7.1, C8.1, U7.VOC_SAMP, U7.VSTOR; no longer C12.1, C13.1, U3.VOC_SAMP, U3.VSTOR
Other:
- note added: "DNP"

Commit message: committing board sent to fab
Connections:
- net GND: no longer TP2.PP, TP6.PP, TP7.PP, TP8.PP
- net N$43: now also TP8.PP
- net N$61: now also TP6.PP
- net N$62: now also TP2.PP
- net N$63: now also TP7.PP
- net N$65: now also TP3.PP
- net N$66: no longer TP1.PP, TP3.PP, TP4.PP
- net N$67: now also TP4.PP
- net N$68: now also TP1.PP
Other:
- moved on the sheet: TP1, TP2, TP3, TP4, TP5, TP6, TP7, TP8
