File: hardware/prototype/rev_B/cinamin.sch (EAGLE design)
At the start: 45 parts, among them U1 AP4400_3.4_2.3, U6 AP4400_3.4_2.3, X1 16Mhz, X3 16Mhz

Commit message: prototype board mostly done, clean up board and schematic before ordering tonight
Parts:
- removed A3: AH212M, chips:AH212M
- removed C7: 1pF, passives:CAPACITOR
- removed PV_TO_CAP, VCC_SELECTOR: (no value), SparkFun-Connectors:M03PTH
- removed R2: 2.2k, passives:RESISTOR0402_RES
- removed U$2: DA14581-40, chips:DA14581-40
- removed U$3: DA14581-BGA, chips:DA14581-BGA
- removed U$4: (no value), chips:LD391151.4V
- removed X3: 16Mhz, crystals:TXC-8Y
- added CM1, CM2: (no value), SparkFun-Passives:JUMPER-2PTH
- added TP10, TP11, TP13, TP14, TP9, VCAP, VIN, VPP, VREG: TPSPAD1-13, testpad:TPSPAD1-13
- C1: value 15uF -> 1pF
- C2: value 15uF -> 1uF
- C3, C4: value 100uF -> 15uF; device passives:CAP_POL0603 -> passives:CAPACITOR
- C5, C6: value 1uF -> 100uF; device passives:CAPACITOR -> passives:CAP_POL0603
- U1: value AP4400_3.4_2.3 -> DA14581-40; device chips:AP4400 -> chips:DA14581-40
- renumbered RESET1 to RESET, U$1 to U2, U6 to U3
Connections:
- removed net DA_VCC: RESET.P$2, U$2.VBAT3V, U$2.VBAT_RF, U2.EN, U2.IN, VCC_SELECTOR.2
- removed net N$10: C6.1, U$3.VDCDC, U$3.VDCDC_RF, U$4.OUT
- removed net N$5: U$3.XTAL16MP, X1.2
- removed net N$6: U$3.VBAT3V, U$3.VBAT_RF, U$4.EN, U$4.IN, U1.DETOUT
- removed net N$66: D1PV.1, D2PV.1, D3PV.1, D4.V+, PV_TO_CAP.2, TP5.PP
- removed net N$8: A1.ANTENNA, U$3.RFIOP
- removed net PV: PV_TO_CAP.1
- net GND: now also C3.2, C4.2, C5.ANODE, C6.ANODE, TP10.PP, TP11.PP, TP13.PP, TP14.PP, TP9.PP, U1.RFIOM, U1.VBAT1V; no longer C3.ANODE, C4.ANODE, C5.2, C6.2, C7.2, R2.1, U$2.GND, U$2.RFIOM, U$2.VBAT1V, U$3.RFIOM, U$3.VBAT1V, U$4.GND, X3.GND
- net N$1: now also C3.1, C4.1, C5.CATHODE, C6.CATHODE, CM1.1, D1PV.1, D2PV.1, D3PV.1, D4.V+, TP5.PP, VCAP.PP; no longer C1.1, C2.1, C3.CATHODE, C4.CATHODE, PV_TO_CAP.3, U3.VDD
- net N$15: now also U1.XTAL16MP, X1.2; no longer U$2.XTAL16MP, X3.2
- net N$18: now also U1.XTAL16MM, X1.1; no longer U$2.XTAL16MM, X3.1
- net N$19: now also A1.ANTENNA, C1.1, U1.RFIOP; no longer A3.ANTENNA, C7.1, U$2.RFIOP
- net N$2: now also U1.VPP, VPP.PP; no longer R2.2, U$3.RST
- net N$22: now also U1.RST; no longer U$2.RST
- net N$3: now also C2.1, U1.VDCDC, U1.VDCDC_RF, VREG.PP; no longer C5.1, U$2.VDCDC, U$2.VDCDC_RF
- net N$4: now also CM2.1, VIN.PP; no longer VCC_SELECTOR.1
- net N$7: now also CM1.2, U3.VDD; no longer U$3.XTAL16MM, X1.1
- net SWDIO: now also U1.SWDIO; no longer U$2.SWDIO, U$3.SWDIO
- net SW_CLK: now also U1.SW_CLK; no longer U$2.SW_CLK, U$3.SW_CLK
- net VCC_EXT: now also CM2.2, RESET.P$2, U1.VBAT3V, U1.VBAT_RF, U2.EN, U2.IN; no longer VCC_SELECTOR.3
Other:
- moved on the sheet: A1, C1, C2, X1

Commit message: prototype to production
Parts:
- removed CM1: (no value), SparkFun-Passives:JUMPER-2PTH
- removed D2-3S, D3-4S: SER, SparkFun-Passives:JUMPER-2PTH
- removed D3PV: HIGH, SparkFun-Passives:JUMPER-2PTH
- removed VCAP, VIN, VREG: TPSPAD1-13, testpad:TPSPAD1-13
- added JP11: CURRENT_MEASURE1, SparkFun-Passives:JUMPER-2PTH
- added JP5: SER2, SparkFun-Passives:JUMPER-2PTH
- added JP7: PAR3, SparkFun-Passives:JUMPER-2PTH
- added JP8: SER3, SparkFun-Passives:JUMPER-2PTH
- added TP12: VCAP, testpad:TPSPAD1-13
- added TP15: VDET, testpad:TPSPAD1-13
- added TP16: VREG, testpad:TPSPAD1-13
- JP1: value HIGH -> PAR1
- JP10: value GND -> GND4
- JP12: value (none) -> CURRENT_MEASURE2
- JP2: value SER -> SER1
- JP3: value GND -> GND1
- JP4: value HIGH -> PAR2
- JP6: value GND -> GND2
- JP9: value GND -> GND3
- TP1: value TPSPAD1-13 -> D3H
- TP10, TP11, TP13, TP14, TP9: value TPSPAD1-13 -> GND
- TP17: value TPSPAD1-13 -> VPP
- TP2: value TPSPAD1-13 -> D2L
- TP3: value TPSPAD1-13 -> D1H
- TP4: value TPSPAD1-13 -> D2H
- TP5: value TPSPAD1-13 -> D4H
- TP6: value TPSPAD1-13 -> D1L
- TP7: value TPSPAD1-13 -> D3L
- TP8: value TPSPAD1-13 -> D4L
- U2: value (none) -> LD391151.4V
- renumbered CM2 to JP12, D1-2S to JP2, D1G to JP3, D1PV to JP1, D2G to JP6, D2PV to JP4, D3G to JP9, D4G to JP10, VPP to TP17
Connections:
- removed net N$4: JP12.1, U3.DETOUT, VIN.PP
- removed net N$43: D3-4S.2, D4.V-, JP10.2, TP8.PP
- removed net N$7: CM1.2, U3.VDD
- new net DET_OUT: JP12.1, TP15.PP, U3.DETOUT
- new net JP10: D4.V-, JP10.2, JP8.2, TP8.PP
- new net VCAP: JP11.2, U3.VDD
- net N$1: now also JP11.1, JP7.1, TP12.PP; no longer CM1.1, D3PV.1, VCAP.PP
- net N$3: now also TP16.PP; no longer VREG.PP
- net N$63: now also JP5.2; no longer D2-3S.2
- net N$67: now also JP5.1; no longer D2-3S.1
- net N$68: now also JP7.2, JP8.1; no longer D3-4S.1, D3PV.2
Other:
- note added: "CURRENT MEASURE"
- note added: "GND Test Pins"
- note added: "Programming"
- note added: "VCAP"
- note added: "VDET"
- note added: "VPP"
- note added: "VREG"
- note added: "Voltage Detector"
- moved on the sheet: TP10, TP11, TP13, TP14, TP6, TP9, U3
