File: hardware/rev_A/cinamin.sch (EAGLE design)
At the start: 11 parts, among them U1 AP4400_3.4_2.3, X1 16Mhz

Commit message: cleaned up some traces, changed to 0603 cap
Parts:
- C1: value 15uF -> 47uF; device passives:CAPACITOR -> passives:CAP_POL0603_SMALL
- U$4: value (none) -> LD391151.4V
Connections:
- net GND: now also C1.ANODE; no longer C1.2
- net N$3: now also C1.CATHODE; no longer C1.1
Changed lines of the file:
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@@
 <part name="FRAME1" library="frames" deviceset="LETTER_L" device=""/>
 <part name="D1" library="chips" deviceset="CPC1822" device="" value="CPC1822"/>
-<part name="C1" library="passives" deviceset="CAPACITOR" device="" value="15uF"/>
 <part name="PROG1" library="connector" deviceset="TC2030-JLINK" device="-L"/>
 <part name="GND23" library="SparkFun-Aesthetics" deviceset="GND" device=""/>
@@
 <part name="TP1" library="testpad" deviceset="TPS" device="PAD1-13"/>
 <part name="TP2" library="testpad" deviceset="TPS" device="PAD1-13"/>
+<part name="C1" library="passives" deviceset="CAP_POL" device="0603_SMALL" value="47uF"/>
 </parts>
 <sheets>
@@
 <instance part="FRAME1" gate="G$2" x="147.32" y="0"/>
 <instance part="D1" gate="G$1" x="15.24" y="99.06"/>
-<instance part="C1" gate="G$1" x="30.48" y="101.6"/>
 <instance part="PROG1" gate="G$1" x="25.4" y="20.32"/>
 <instance part="GND23" gate="1" x="7.62" y="7.62"/>
@@
 <instance part="TP1" gate="G$1" x="73.66" y="86.36"/>
 <instance part="TP2" gate="G$1" x="33.02" y="66.04"/>
+<instance part="C1" gate="G$1" x="30.48" y="99.06"/>
 </instances>
 <busses>
@@
 <wire x1="15.24" y1="86.36" x2="30.48" y2="86.36" width="0.1524" layer="91"/>
 <junction x="50.8" y="86.36"/>
-<pinref part="C1" gate="G$1" pin="2"/>
 <wire x1="30.48" y1="86.36" x2="50.8" y2="86.36" width="0.1524" layer="91"/>
 <wire x1="30.48" y1="96.52" x2="30.48" y2="86.36" width="0.1524" layer="91"/>
 <junction x="30.48" y="86.36"/>
+<pinref part="C1" gate="G$1" pin="ANODE"/>
 </segment>
 <segment>
@@
 <wire x1="30.48" y1="119.38" x2="50.8" y2="119.38" width="0.1524" layer="91"/>
 <wire x1="50.8" y1="119.38" x2="50.8" y2="114.3" width="0.1524" layer="91"/>
-<pinref part="C1" gate="G$1" pin="1"/>
-<wire x1="30.48" y1="104.14" x2="30.48" y2="119.38" width="0.1524" layer="91"/>
+<wire x1="30.48" y1="101.6" x2="30.48" y2="119.38" width="0.1524" layer="91"/>
 <junction x="30.48" y="119.38"/>
-</segment>
-</net>
+<pinref part="C1" gate="G$1" pin="CATHODE"/>
+</segment>
+</net>
